File: Circuits/Boards R3/Swarm Board_3.brd (EAGLE design)
At the start: 56.1 x 63.5 mm, 103 parts, among them CON1 ISP(2X3), CON3 MAINCONNECTOR_16SMD, CON4 HEADER_3X1, CON5 HEADER_3X1, CON6 MAIN_CONNECTOR_10SMD, T1 NPN2N2222, T10 TEFT4300, T11 NPN2N2222, T13 NPN2N2222, T14 NPN2N2222, T15 NPN2N2222, T16 NPN2N2222, T17 NPN2N2222, T18 NPN2N2222, T2 NPN2N2222, T3 NPN2N2222, T4 TEFT4300, T5 TEFT4300, T6 TEFT4300, T7 TEFT4300, T8 TEFT4300, T9 TEFT4300, U1 ATMEGA324P, U2 MCP73833, U3 ATMEGA1281, U4 MCP9700A, U5 AH182, U6 AH182

Commit message: R3 Work
Parts:
- removed CON3: MAINCONNECTOR_16SMD, Mechanical:FEMALE_HEADER_2MM_2X8_SMD
- removed CON6: MAIN_CONNECTOR_10SMD, Mechanical:FEMALE_HEADER_2MM_2X5_SMD
- added C15, C4: 1uf, Passive:0603
- added CON2: MAIN_CONNECTOR_14SMD, Mechanical:FEMALE_HEADER_2MM_2X7_SMD
- added CON7: MAIN_CONNECTOR_8, Mechanical:FEMALE_HEADER_2MM_2X4
- added LED11, LED12, LED14, LED15: (no value), Passive:LED0603
- added LED8, LED9: IR, Passive:5MM_LED_RA
- added R26, R43, R48, R49: 10k, Passive:0603
- added R44, R45: 4.7k, Passive:0603
- added R46, R47, R52: 100, Passive:0603
- added R50, R51: 220, Passive:0603
- added R53, R54, R55, R56: 1k, Passive:0603
- added T12: SI2333DS-T1, Passive:SOT23
- added T19, T20, T21, T22: IRLML6244TR, Passive:SOT23
- added U7, U8, U9: QRE1113, Passive:QRE1113
- C7: value 10uf -> 1uf; device Passive:0805 -> Passive:0603
- R33, R34, R35: value 20k -> 22k
- T1, T2: value NPN2N2222 -> TEFT4300; device Passive:SOT23 -> Passive:3MM_LED_RA
- moved ANT4 92.9 mm to (36.0, 50.8), flipped to the bottom
- moved U6 89.0 mm to (50.2, 39.4), turned to 270 degrees
- moved R2 82.4 mm to (88.4, 32.6)
- moved C14 75.3 mm to (84.6, 34.9), turned to 180 degrees
- moved T11 72.0 mm to (46.8, 10.7), turned to 225 degrees
- moved B1 63.1 mm to (23.5, 70.9)
- moved R28 63.1 mm to (23.6, 75.9)
- moved R8 63.1 mm to (23.7, 69.0)
- moved C1 57.2 mm to (75.3, 35.8)
- moved C13 57.2 mm to (71.5, 35.8)
- moved C2 57.2 mm to (77.0, 30.1)
- moved CON4 57.2 mm to (78.5, 44.1)
- moved R30 57.2 mm to (73.4, 35.8)
- moved R31 57.2 mm to (69.6, 35.8)
- moved R32 57.2 mm to (67.7, 35.8)
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Connections:
- removed net EM: CON3.13
- removed net EMSENSE: CON3.14
- removed net SEM: CON6.7
- removed net SEMSENSE: CON6.6
- removed net VSENSE: R29.1, R30.2, U1.37
- new net +VSENSE: C4.1, C5.1, CON2.6, PR1.2, R25.2, R36.2, R37.2, R38.2, R39.2, R40.2, R41.2, R44.2, R45.2, R6.2, T1.1, T10.1, T12.3, T2.1, T4.1, T5.1, T6.1, T7.1, T8.1, T9.1, U4.1, U5.1, U6.1
- new net LED4: R53.1, R54.1, R55.1, R56.1
- new net N$20: LED8.2, R46.2
- new net N$21: LED9.2, R47.2
- new net N$29: R51.1, U7.P$2
- new net N$3: R43.2, T11.1, T2.2
- new net N$39: R50.1, U8.P$2
- new net N$40: R48.1
- new net N$41: R49.1
- new net N$42: R52.1, U9.P$2
- new net N$43: LED11.1, R53.2
- new net N$45: LED12.1, R54.2
- new net N$46: LED14.1, R55.2
- new net N$47: LED15.1, R56.2
- new net N$6: R26.2, T1.2, T3.1
- new net RX7: R44.1, T3.3
- new net RX8: R45.1, T11.3
- new net SEN: T12.1
- new net VBATSENSE: C15.1, R29.1, R30.2, U1.37
- net +3V: now also LED11.2, LED12.2, LED14.2, LED15.2, LED8.1, LED9.1, T12.2; no longer C5.1, CON3.7, PR1.2, R25.2, R36.2, R37.2, R38.2, R39.2, R40.2, R41.2, R6.2, T10.1, T4.1, T5.1, T6.1, T7.1, T8.1, T9.1, U4.1, U5.1, U6.1
- net GND: now also C15.2, C4.2, CON2.8, CON2.9, R26.1, R43.1, T11.2, T19.2, T20.2, T21.2; no longer CON3.10, CON3.9, T1.2, T2.2
- net IRBUMBER: now also CON2.12; no longer CON3.5
- net IRENABLE: now also CON2.5; no longer CON3.6
- net LEFTBUMPER: now also CON2.11; no longer CON3.12
- net LINESENSE1: now also CON2.4; no longer CON3.3
- net LINESENSE2: now also CON2.3; no longer CON3.4
- net MA+: now also CON2.13; no longer CON3.15
- net MA-: now also CON2.14; no longer CON3.16
- net MB+: now also CON2.2; no longer CON3.2
- net MB-: now also CON2.1; no longer CON3.1
- net N$10: now also R46.1, R47.1, T21.3; no longer T2.3
- net N$11: now also T21.1; no longer T2.1
- net N$12: now also T20.3; no longer T3.3
- net N$19: now also T20.1; no longer T3.1
- net N$2: now also R50.2, R51.2, R52.2, T22.3; no longer T11.3
- net N$26: now also T19.1; no longer T1.1
- net N$4: now also T22.1; no longer T11.1
- net N$5: now also CON2.7; no longer CON3.8
- net N$9: now also T19.3; no longer T1.3
- net RIGHTBUMPER: now also CON2.10; no longer CON3.11
- net S3V: now also CON7.1, R48.2, R49.2, U7.P$1, U7.P$3, U8.P$1, U8.P$3, U9.P$1, U9.P$3; no longer CON6.1
- net SGND: now also CON7.8, T22.2; no longer CON6.10, T11.2
- net SIRBUMPER: now also CON7.5, U9.P$4; no longer CON6.3
- net SIRENABLE: now also CON7.2; no longer CON6.2
- net SLEFTBUMPER: now also CON7.6; no longer CON6.8
- net SLINESENSE1: now also CON7.3, U8.P$4; no longer CON6.5
- net SLINESENSE2: now also CON7.4; no longer CON6.4
- net SLINSENSE2: now also U7.P$4
- net SRIGHTBUMPER: now also CON7.7; no longer CON6.9
Routing:
- net +3V: track 362.5 -> 19.6 mm, vias 7 -> 0
- net N$10: track 172.3 -> 1.10 mm
- net RX1: track 47.1 -> 0.00 mm, vias 2 -> 0
- net +VRAW: track 85.7 -> 39.7 mm, vias 7 -> 5
- net DISTANCERECEIVE: track 48.9 -> 3.40 mm, vias 2 -> 0
- net RX3: track 42.7 -> 1.96 mm, vias 2 -> 0
- net DISTANCELED: track 39.7 -> 0.00 mm, vias 2 -> 0
- net CHGSTATUS: track 43.4 -> 3.85 mm
- net TRANSMITLEDS: track 38.2 -> 0.00 mm, vias 2 -> 0
- net CHGDETECT: track 39.5 -> 2.05 mm
- net GND: track 90.6 -> 53.3 mm, vias 16 -> 9
- net RX2: track 37.8 -> 2.10 mm, vias 2 -> 0
- net IRENABLE: track 34.5 -> 0.00 mm, vias 2 -> 0
- net RX6: track 36.1 -> 2.10 mm, vias 4 -> 0
- net RX4: track 35.9 -> 2.05 mm, vias 2 -> 0
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
Commit message: More R3 work
Parts:
- added C16: 1uf, Passive:0603
- added M1: VIBMOTOR, Mechanical:VIBMOTOR
- added R57: 0, Passive:0603
- added R58: 1k, Passive:0603
- added T23: IRLML6244TR, Passive:SOT23
- R22: value 15 -> 32
- R29: value 7.5k -> 100k
- R30: value 18k -> 100k
- moved T12 139.0 mm to (69.7, 52.1)
- moved H1 14.0 mm to (6.35, 39.4)
- moved U5 7.01 mm to (6.35, 24.7)
Connections:
- net S3V renamed S+VSENSE
- new net N$44: R58.2, T23.1
- new net N$48: M1.P$2, R57.2
- new net N$7: R57.1, T23.3
- net +VCHG: now also ANT1.P$2
- net +VRAW: now also C16.1, M1.P$1
- net DISTANCELED: now also R58.1
- net GND: now also ANT3.P$2, C16.2, T23.2
- net SCL: now also ANT4.P$2
- net SDA: now also ANT2.P$2
