File: Circuits/Boards R3/Swarm Board_3.sch (EAGLE design)
At the start: 103 parts, among them CON1 ISP(2X3), CON3 MAINCONNECTOR_16SMD, CON4 HEADER_3X1, CON5 HEADER_3X1, CON6 MAIN_CONNECTOR_10SMD, T1 NPN2N2222, T10 TEFT4300, T11 NPN2N2222, T13 NPN2N2222, T14 NPN2N2222, T15 NPN2N2222, T16 NPN2N2222, T17 NPN2N2222, T18 NPN2N2222, T2 NPN2N2222, T3 NPN2N2222, T4 TEFT4300, T5 TEFT4300, T6 TEFT4300, T7 TEFT4300, T8 TEFT4300, T9 TEFT4300, U1 ATMEGA324P, U2 MCP73833, U3 ATMEGA1281, U4 MCP9700A, U5 AH182, U6 AH182

Commit message: R3 Work
Parts:
- removed CON3: MAINCONNECTOR_16SMD, Mechanical:MAINCONNECTOR_16SMD
- removed CON6: MAIN_CONNECTOR_10SMD, Mechanical:MAIN_CONNECTOR_10SMD
- added C15, C4: 1uf, Passive:CAP0603
- added CON2: MAIN_CONNECTOR_14SMD, Mechanical:MAIN_CONNECTOR_14SMD
- added CON7: MAIN_CONNECTOR_8, Mechanical:MAIN_CONNECTOR_8
- added LED11, LED12, LED14, LED15: (no value), Passive:LED0603
- added LED8, LED9: IR, Passive:LED5MMRA
- added R26, R43, R48, R49: 10k, Passive:RES0603
- added R44, R45: 4.7k, Passive:RES0603
- added R46, R47, R52: 100, Passive:RES0603
- added R50, R51: 220, Passive:RES0603
- added R53, R54, R55, R56: 1k, Passive:RES0603
- added T12: SI2333DS-T1, Passive:SI2333DS-T1
- added T19, T20, T21, T22: IRLML6244TR, Passive:IRLML6244TR
- added U7, U8, U9: QRE1113, Passive:QRE1113
- C7: value 10uf -> 1uf; device Passive:CAP0805 -> Passive:CAP0603
- R33, R34, R35: value 20k -> 22k
- T1, T2: value NPN2N2222 -> TEFT4300; device Passive:NPN2N2222 -> Passive:TEFT4300
Connections:
- removed net EM: CON3.13
- removed net EMSENSE: CON3.14
- removed net SEM: CON6.7
- removed net SEMSENSE: CON6.6
- removed net VSENSE: R29.1, R30.2, U1.PA0(ADC0/PCINT0)
- new net +VSENSE: C4.1, C5.1, CON2.6, PR1.2, R25.2, R36.2, R37.2, R38.2, R39.2, R40.2, R41.2, R44.2, R45.2, R6.2, T1.C, T10.C, T12.D, T2.C, T4.C, T5.C, T6.C, T7.C, T8.C, T9.C, U4.VCC, U5.VCC, U6.VCC
- new net LED4: R53.1, R54.1, R55.1, R56.1
- new net N$20: LED8.C, R46.2
- new net N$21: LED9.C, R47.2
- new net N$29: R51.1, U7.CT
- new net N$3: R43.2, T11.B, T2.E
- new net N$39: R50.1, U8.CT
- new net N$40: R48.1
- new net N$41: R49.1
- new net N$42: R52.1, U9.CT
- new net N$43: LED11.C, R53.2
- new net N$45: LED12.C, R54.2
- new net N$46: LED14.C, R55.2
- new net N$47: LED15.C, R56.2
- new net N$6: R26.2, T1.E, T3.B
- new net RX7: R44.1, T3.C
- new net RX8: R45.1, T11.C
- new net SEN: T12.G
- new net VBATSENSE: C15.1, R29.1, R30.2, U1.PA0(ADC0/PCINT0)
- net +3V: now also LED11.A, LED12.A, LED14.A, LED15.A, LED8.A, LED9.A, T12.S; no longer C5.1, CON3.7, PR1.2, R25.2, R36.2, R37.2, R38.2, R39.2, R40.2, R41.2, R6.2, T10.C, T4.C, T5.C, T6.C, T7.C, T8.C, T9.C, U4.VCC, U5.VCC, U6.VCC
- net GND: now also C15.2, C4.2, CON2.8, CON2.9, R26.1, R43.1, T11.E, T19.S, T20.S, T21.S; no longer CON3.10, CON3.9, T1.E, T2.E
- net IRBUMBER: now also CON2.12; no longer CON3.5
- net IRENABLE: now also CON2.5; no longer CON3.6
- net LEFTBUMPER: now also CON2.11; no longer CON3.12
- net LINESENSE1: now also CON2.4; no longer CON3.3
- net LINESENSE2: now also CON2.3; no longer CON3.4
- net MA+: now also CON2.13; no longer CON3.15
- net MA-: now also CON2.14; no longer CON3.16
- net MB+: now also CON2.2; no longer CON3.2
- net MB-: now also CON2.1; no longer CON3.1
- net N$10: now also R46.1, R47.1, T21.D; no longer T2.C
- net N$11: now also T21.G; no longer T2.B
- net N$12: now also T20.D; no longer T3.C
- net N$19: now also T20.G; no longer T3.B
- net N$2: now also R50.2, R51.2, R52.2, T22.D; no longer T11.C
- net N$26: now also T19.G; no longer T1.B
- net N$4: now also T22.G; no longer T11.B
- net N$5: now also CON2.7; no longer CON3.8
- net N$9: now also T19.D; no longer T1.C
- net RIGHTBUMPER: now also CON2.10; no longer CON3.11
- net S3V: now also CON7.1, R48.2, R49.2, U7.AN, U7.C, U8.AN, U8.C, U9.AN, U9.C; no longer CON6.1
- net SGND: now also CON7.8, T22.S; no longer CON6.10, T11.E
- net SIRBUMPER: now also CON7.5, U9.E; no longer CON6.3
- net SIRENABLE: now also CON7.2; no longer CON6.2
- net SLEFTBUMPER: now also CON7.6; no longer CON6.8
- net SLINESENSE1: now also CON7.3, U8.E; no longer CON6.5
- net SLINESENSE2: now also CON7.4; no longer CON6.4
- net SLINSENSE2: now also U7.E
- net SRIGHTBUMPER: now also CON7.7; no longer CON6.9
Other:
- note added: "CHANGE DIVIDER VALUES"
- moved on the sheet: ANT1, ANT2, ANT3, ANT4, C10, C11, C14, C3, C5, C7, C8, C9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

Commit message: More R3 work
Parts:
- added C16: 1uf, Passive:CAP0603
- added M1: VIBMOTOR, Mechanical:VIBMOTOR
- added R57: 0, Passive:RES0603
- added R58: 1k, Passive:RES0603
- added T23: IRLML6244TR, Passive:IRLML6244TR
- R22: value 15 -> 32
- R29: value 7.5k -> 100k
- R30: value 18k -> 100k
Connections:
- net S3V renamed S+VSENSE
- new net N$44: R58.2, T23.G
- new net N$48: M1.-VM, R57.2
- new net N$7: R57.1, T23.D
- net +VRAW: now also C16.1, M1.+VM
- net DISTANCELED: now also R58.1
- net GND: now also C16.2, T23.S
Other:
- note added: "maybe replace ir bumper with +3v?"
- moved on the sheet: ANT1, ANT2, ANT3, ANT4
Changed lines of the file:
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@@
 <part name="C6" library="Passive" deviceset="CAP" device="0805" value="10uf"/>
 <part name="P+9" library="Supply" deviceset="+3V" device=""/>
-<part name="R22" library="Passive" deviceset="RES" device="0603" value="15"/>
+<part name="R22" library="Passive" deviceset="RES" device="0603" value="32"/>
 <part name="R23" library="Passive" deviceset="RES" device="0603" value="1k"/>
 <part name="GND9" library="Supply" deviceset="GND" device=""/>
@@
 <part name="R41" library="Passive" deviceset="RES" device="0603" value="4.7k"/>
 <part name="U2" library="PowerIC" deviceset="MCP73833" device=""/>
-<part name="R29" library="Passive" deviceset="RES" device="0603" value="7.5k"/>
-<part name="R30" library="Passive" deviceset="RES" device="0603" value="18k"/>
+<part name="R29" library="Passive" deviceset="RES" device="0603" value="100k"/>
+<part name="R30" library="Passive" deviceset="RES" device="0603" value="100k"/>
 <part name="R31" library="Passive" deviceset="RES" device="0603" value="10k"/>
 <part name="R32" library="Passive" deviceset="RES" device="0603" value="2k"/>
@@
 <part name="P+17" library="Supply" deviceset="+3V" device=""/>
 <part name="C7" library="Passive" deviceset="CAP" device="0603" value="1uf"/>
+<part name="R57" library="Passive" deviceset="RES" device="0603" value="0"/>
+<part name="R58" library="Passive" deviceset="RES" device="0603" value="1k"/>
+<part name="GND24" library="Supply" deviceset="GND" device=""/>
+<part name="T23" library="Passive" deviceset="IRLML6244TR" device=""/>
+<part name="C16" library="Passive" deviceset="CAP" device="0603" value="1uf"/>
+<part name="P+21" library="Supply" deviceset="+VRAW" device=""/>
+<part name="M1" library="Mechanical" deviceset="VIBMOTOR" device=""/>
 </parts>
 <sheets>
@@
 <text x="-76.2" y="2.54" size="1.778" layer="97">PICK NEW 8MHX XTAL</text>
 <text x="-76.2" y="73.66" size="1.778" layer="97">CHANGE DIVIDER VALUES</text>
+<text x="370.84" y="-86.36" size="1.778" layer="97">maybe replace ir bumper with +3v?</text>
 </plain>
 <instances>
@@
 <instance part="P+17" gate="1" x="-76.2" y="-22.86" rot="MR0"/>
 <instance part="C7" gate="G$1" x="165.1" y="-10.16"/>
+<instance part="R57" gate="G$1" x="-160.02" y="-116.84" rot="R90"/>
+<instance part="R58" gate="G$1" x="-175.26" y="-134.62"/>
+<instance part="GND24" gate="1" x="-160.02" y="-147.32"/>
+<instance part="T23" gate="G$1" x="-162.56" y="-132.08"/>
+<instance part="C16" gate="G$1" x="-149.86" y="-127"/>
+<instance part="P+21" gate="G$1" x="-149.86" y="-93.98" rot="MR0"/>
+<instance part="M1" gate="G$1" x="-167.64" y="-104.14" rot="MR0"/>
 </instances>
 <busses>
@@
 <junction x="434.34" y="66.04"/>
 </segment>
+<segment>
+<wire x1="-160.02" y1="-137.16" x2="-160.02" y2="-142.24" width="0.1524" layer="91"/>
+<pinref part="GND24" gate="1" pin="GND"/>
+<wire x1="-160.02" y1="-142.24" x2="-160.02" y2="-144.78" width="0.1524" layer="91"/>
+<wire x1="-160.02" y1="-142.24" x2="-149.86" y2="-142.24" width="0.1524" layer="91"/>
+<wire x1="-149.86" y1="-142.24" x2="-149.86" y2="-129.54" width="0.1524" layer="91"/>
+<junction x="-160.02" y="-142.24"/>
+<pinref part="T23" gate="G$1" pin="S"/>
+<pinref part="C16" gate="G$1" pin="2"/>
+</segment>
 </net>
 <net name="+VBAT" class="0">
@@
 <label x="58.42" y="-193.04" size="1.778" layer="91" xref="yes"/>
 </segment>
+<segment>
+<pinref part="R58" gate="G$1" pin="1"/>
+<wire x1="-180.34" y1="-134.62" x2="-185.42" y2="-134.62" width="0.1524" layer="91"/>
+<label x="-185.42" y="-134.62" size="1.778" layer="91" rot="R180" xref="yes"/>
+</segment>
 </net>
 <net name="STBY" class="0">
@@
 <pinref part="P+20" gate="G$1" pin="+VRAW"/>
 <wire x1="-132.08" y1="-22.86" x2="-132.08" y2="-25.4" width="0.1524" layer="91"/>
+</segment>
+<segment>
+<wire x1="-162.56" y1="-99.06" x2="-149.86" y2="-99.06" width="0.1524" layer="91"/>
+<wire x1="-149.86" y1="-99.06" x2="-149.86" y2="-121.92" width="0.1524" layer="91"/>
+<wire x1="-149.86" y1="-99.06" x2="-149.86" y2="-93.98" width="0.1524" layer="91"/>
+<junction x="-149.86" y="-99.06"/>
+<pinref part="C16" gate="G$1" pin="1"/>
+<pinref part="P+21" gate="G$1" pin="+VRAW"/>
+<pinref part="M1" gate="G$1" pin="+VM"/>
 </segment>
 </net>
@@
 <wire x1="449.58" y1="-154.94" x2="449.58" y2="-157.48" width="0.1524" layer="91"/>
 <label x="449.58" y="-157.48" size="1.778" layer="91" rot="R270" xref="yes"/>
+<junction x="449.58" y="-154.94"/>
 </segment>
 </net>
@@
 </segment>
 </net>
-<net name="S3V" class="0">
+<net name="S+VSENSE" class="0">
 <segment>
 <pinref part="C14" gate="G$1" pin="1"/>
@@
 </segment>
 </net>
+<net name="DEBUG1" class="0">
+<segment>
+<wire x1="-63.5" y1="-48.26" x2="-63.5" y2="-50.8" width="0.1524" layer="91"/>
+<label x="-63.5" y="-50.8" size="1.778" layer="91" rot="R270" xref="yes"/>
+</segment>
+</net>
+<net name="DEBUG2" class="0">
+<segment>
+<wire x1="-53.34" y1="-48.26" x2="-53.34" y2="-50.8" width="0.1524" layer="91"/>
+<label x="-53.34" y="-50.8" size="1.778" layer="91" rot="R270" xref="yes"/>
+</segment>
+</net>
+<net name="N$7" class="0">
+<segment>
+<pinref part="R57" gate="G$1" pin="1"/>
+<wire x1="-160.02" y1="-121.92" x2="-160.02" y2="-127" width="0.1524" layer="91"/>
+<pinref part="T23" gate="G$1" pin="D"/>
+</segment>
+</net>
+<net name="N$44" class="0">
+<segment>
+<pinref part="R58" gate="G$1" pin="2"/>
+<wire x1="-170.18" y1="-134.62" x2="-165.1" y2="-134.62" width="0.1524" layer="91"/>
+<pinref part="T23" gate="G$1" pin="G"/>
+</segment>
+</net>
+<net name="N$48" class="0">
+<segment>
+<pinref part="R57" gate="G$1" pin="2"/>
+<wire x1="-160.02" y1="-111.76" x2="-160.02" y2="-109.22" width="0.1524" layer="91"/>
+<pinref part="M1" gate="G$1" pin="-VM"/>
+<wire x1="-160.02" y1="-109.22" x2="-162.56" y2="-109.22" width="0.1524" layer="91"/>
+</segment>
+</net>
 </nets>
 </sheet>
 </sheets>
+<errors>
+</errors>
 </schematic>
 </drawing>
